File: eagle/nek-type-a/left.brd (EAGLE design)
At the start: 133 x 116 mm, 69 parts

Commit message: left routed
Routing:
- net ROW6: track 0.00 -> 197.4 mm
- net ROW5: track 0.00 -> 175.5 mm
- net ROW4: track 0.00 -> 157.8 mm
- net COL5: track 0.00 -> 155.2 mm
- net COL6: track 0.00 -> 148.3 mm
- net ROW3: track 0.00 -> 134.8 mm
- net COL2: track 0.00 -> 130.6 mm
- net COL3: track 0.00 -> 124.0 mm
- net ROW2: track 0.00 -> 123.0 mm
- net COL4: track 0.00 -> 120.5 mm
- net COL1: track 0.00 -> 120.2 mm
- net ROW1: track 0.00 -> 113.5 mm
- net COL7: track 0.00 -> 99.4 mm
- net N$29: track 0.00 -> 6.52 mm
- net N$28: track 0.00 -> 6.52 mm
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