File: eagle/nek-type-a/left.sch (EAGLE design)
At the start: 68 parts

Commit message: columns
Parts:
- added LEFT: LEFT, con-harting:CON16
Connections:
- net ROW2.25 renamed ROW2
- removed net N$35: CAPSLOCK.P0, CONTROL.P0, SHIFT.P0, TAB.P0, TICK.P0
- removed net N$36: 1.P0, A.P0, ESC.P0, OPTION.P0, Q.P0, Z.P0
- removed net N$37: 2.P0, COMMAND.P0, S.P0, W.P0, X.P0
- removed net N$38: 3.P0, C.P0, D.P0, E.P0, F1.P0
- removed net N$39: 4.P0, F.P0, F2.P0, R.P0, SPACE.P0, V.P0
- removed net N$40: 5.P0, B.P0, F3.P0, G.P0, T.P0
- removed net N$41: 6.P0, F4.P0
- new net COL1: CAPSLOCK.P0, CONTROL.P0, LEFT.2, SHIFT.P0, TAB.P0, TICK.P0
- new net COL2: 1.P0, A.P0, ESC.P0, LEFT.4, OPTION.P0, Q.P0, Z.P0
- new net COL3: 2.P0, COMMAND.P0, LEFT.6, S.P0, W.P0, X.P0
- new net COL4: 3.P0, C.P0, D.P0, E.P0, F1.P0, LEFT.8
- new net COL5: 4.P0, F.P0, F2.P0, LEFT.10, R.P0, SPACE.P0, V.P0
- new net COL6: 5.P0, B.P0, F3.P0, G.P0, LEFT.12, T.P0
- new net COL7: 6.P0, F4.P0, LEFT.14

Commit message: rows connected
Parts:
- LEFT: device con-harting:CON16 -> con-harting:CON14
Connections:
- removed net ROW3.25: DE.C, DQ.C, DR.C, DT.C, DTAB.C, DW.C
- removed net ROW4.25: DA.C, DCAPSLOCK.C, DD.C, DF.C, DG.C, DS.C
- removed net ROW5.25: DB.C, DC.C, DSHIFT.C, DV.C, DX.C, DZ.C
- removed net ROW6.25: DCOMMAND.C, DCONTROL.C, DOPTION.C, DSPACE.C
- new net ROW3: DE.C, DQ.C, DR.C, DT.C, DTAB.C, DW.C, LEFT.5
- new net ROW4: DA.C, DCAPSLOCK.C, DD.C, DF.C, DG.C, DS.C, LEFT.7
- new net ROW5: DB.C, DC.C, DSHIFT.C, DV.C, DX.C, DZ.C, LEFT.9
- new net ROW6: DCOMMAND.C, DCONTROL.C, DOPTION.C, DSPACE.C, LEFT.11
- net ROW1: now also LEFT.1
- net ROW2: now also LEFT.3
Changed lines of the file:
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@@
 <part name="SPACE" library="Keyboard" deviceset="KEYSWITCH-PLAIN" device="-MX-2U"/>
 <part name="DSPACE" library="Controller" deviceset="DIODE" device="-DO-35" value="1N4148"/>
-<part name="LEFT" library="con-harting" library_urn="urn:adsk.eagle:library:151" deviceset="CON16" device="" package3d_urn="urn:adsk.eagle:package:7118/1" value="LEFT"/>
+<part name="LEFT" library="con-harting" library_urn="urn:adsk.eagle:library:151" deviceset="CON14" device="" package3d_urn="urn:adsk.eagle:package:7117/1" value="LEFT"/>
 </parts>
 <sheets>
@@
 <instance part="SPACE" gate="G$1" x="106.934" y="-218.948"/>
 <instance part="DSPACE" gate="D$1" x="109.474" y="-203.708" rot="R90"/>
-<instance part="LEFT" gate="G$1" x="-17.78" y="-38.1" rot="R180"/>
+<instance part="LEFT" gate="G$1" x="-17.78" y="-35.56" rot="R180"/>
 </instances>
 <busses>
@@
 <wire x1="102.362" y1="1.27" x2="121.412" y2="1.27" width="0.1524" layer="91"/>
 <junction x="102.362" y="1.27"/>
+<pinref part="LEFT" gate="G$1" pin="1"/>
+<wire x1="-25.4" y1="-27.94" x2="-25.4" y2="0" width="0.1524" layer="91"/>
+<wire x1="-25.4" y1="0" x2="28.702" y2="1.27" width="0.1524" layer="91"/>
+<junction x="28.702" y="1.27"/>
+<label x="127" y="2.54" size="1.778" layer="91" xref="yes"/>
 </segment>
 </net>
@@
 <wire x1="107.188" y1="-46.228" x2="126.238" y2="-46.228" width="0.1524" layer="91"/>
 <junction x="107.188" y="-46.228"/>
-</segment>
-</net>
-<net name="ROW3.25" class="0">
+<wire x1="11.938" y1="-46.228" x2="-27.94" y2="-53.34" width="0.1524" layer="91"/>
+<junction x="11.938" y="-46.228"/>
+<pinref part="LEFT" gate="G$1" pin="3"/>
+<wire x1="-25.4" y1="-30.48" x2="-27.94" y2="-30.48" width="0.1524" layer="91"/>
+<wire x1="-27.94" y1="-30.48" x2="-27.94" y2="-53.34" width="0.1524" layer="91"/>
+<label x="132.08" y="-45.72" size="1.778" layer="91" xref="yes"/>
+</segment>
+</net>
+<net name="ROW3" class="0">
 <segment>
 <pinref part="DTAB" gate="D$1" pin="C"/>
@@
 <wire x1="97.79" y1="-84.328" x2="121.412" y2="-84.328" width="0.1524" layer="91"/>
 <junction x="97.79" y="-84.328"/>
-</segment>
-</net>
-<net name="ROW4.25" class="0">
+<wire x1="16.764" y1="-84.328" x2="-30.48" y2="-86.36" width="0.1524" layer="91"/>
+<junction x="16.764" y="-84.328"/>
+<wire x1="-30.48" y1="-86.36" x2="-30.48" y2="-33.02" width="0.1524" layer="91"/>
+<pinref part="LEFT" gate="G$1" pin="5"/>
+<wire x1="-25.4" y1="-33.02" x2="-30.48" y2="-33.02" width="0.1524" layer="91"/>
+<label x="127" y="-83.82" size="1.778" layer="91" xref="yes"/>
+</segment>
+</net>
+<net name="ROW4" class="0">
 <segment>
 <pinref part="DCAPSLOCK" gate="D$1" pin="C"/>
@@
 <wire x1="102.362" y1="-122.428" x2="123.952" y2="-122.428" width="0.1524" layer="91"/>
 <junction x="102.362" y="-122.428"/>
-</segment>
-</net>
-<net name="ROW5.25" class="0">
+<wire x1="19.05" y1="-122.428" x2="-33.02" y2="-121.92" width="0.1524" layer="91"/>
+<junction x="19.05" y="-122.428"/>
+<wire x1="-33.02" y1="-35.56" x2="-33.02" y2="-101.6" width="0.1524" layer="91"/>
+<pinref part="LEFT" gate="G$1" pin="7"/>
+<wire x1="-25.4" y1="-35.56" x2="-33.02" y2="-35.56" width="0.1524" layer="91"/>
+<wire x1="-33.02" y1="-121.92" x2="-33.02" y2="-101.6" width="0.1524" layer="91"/>
+<label x="129.54" y="-121.92" size="1.778" layer="91" xref="yes"/>
+</segment>
+</net>
+<net name="ROW5" class="0">
 <segment>
 <pinref part="DSHIFT" gate="D$1" pin="C"/>
@@
 <wire x1="107.188" y1="-160.528" x2="126.238" y2="-160.528" width="0.1524" layer="91"/>
 <junction x="107.188" y="-160.528"/>
-</segment>
-</net>
-<net name="ROW6.25" class="0">
+<pinref part="LEFT" gate="G$1" pin="9"/>
+<wire x1="-25.4" y1="-38.1" x2="-35.56" y2="-38.1" width="0.1524" layer="91"/>
+<wire x1="-35.56" y1="-38.1" x2="-35.56" y2="-160.02" width="0.1524" layer="91"/>
+<wire x1="-35.56" y1="-160.02" x2="21.59" y2="-160.528" width="0.1524" layer="91"/>
+<junction x="21.59" y="-160.528"/>
+<label x="132.08" y="-160.02" size="1.778" layer="91" xref="yes"/>
+</segment>
+</net>
+<net name="ROW6" class="0">
 <segment>
 <pinref part="DCONTROL" gate="D$1" pin="C"/>
@@
 <wire x1="69.088" y1="-198.628" x2="109.474" y2="-198.628" width="0.1524" layer="91"/>
 <junction x="69.088" y="-198.628"/>
-</segment>
-</net>
+<wire x1="16.764" y1="-198.628" x2="-38.1" y2="-198.12" width="0.1524" layer="91"/>
+<junction x="16.764" y="-198.628"/>
+<wire x1="-38.1" y1="-198.12" x2="-38.1" y2="-40.64" width="0.1524" layer="91"/>
+<pinref part="LEFT" gate="G$1" pin="11"/>
+<wire x1="-38.1" y1="-40.64" x2="-25.4" y2="-40.64" width="0.1524" layer="91"/>
+<label x="116.84" y="-198.12" size="1.778" layer="91" xref="yes"/>
+</segment>
+</net>

Commit message: move diodes away from stabilizers
Parts:
- LEFTCON: value LEFT -> LEFTCON
- renumbered LEFT to LEFTCON
Changed lines of the file:
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@@
 <drawing>
 <settings>
-<setting alwaysvectorfont="no"/>
+<setting alwaysvectorfont="yes"/>
 <setting verticaltext="up"/>
 </settings>
-<grid distance="0.1" unitdist="inch" unit="inch" style="lines" multiple="1" display="yes" altdistance="0.01" altunitdist="inch" altunit="inch"/>
+<grid distance="0.1" unitdist="inch" unit="inch" style="lines" multiple="1" display="no" altdistance="0.01" altunitdist="inch" altunit="inch"/>
 <layers>
 <layer number="1" name="Top" color="4" fill="1" visible="no" active="no"/>
@@
 <part name="SPACE" library="Keyboard" deviceset="KEYSWITCH-PLAIN" device="-MX-2U"/>
 <part name="DSPACE" library="Controller" deviceset="DIODE" device="-DO-35" value="1N4148"/>
-<part name="LEFT" library="con-harting" library_urn="urn:adsk.eagle:library:151" deviceset="CON14" device="" package3d_urn="urn:adsk.eagle:package:7117/1" value="LEFT"/>
+<part name="LEFTCON" library="con-harting" library_urn="urn:adsk.eagle:library:151" deviceset="CON14" device="" package3d_urn="urn:adsk.eagle:package:7117/1" value="LEFTCON"/>
 </parts>
 <sheets>
@@
 <instance part="SPACE" gate="G$1" x="106.934" y="-218.948"/>
 <instance part="DSPACE" gate="D$1" x="109.474" y="-203.708" rot="R90"/>
-<instance part="LEFT" gate="G$1" x="-17.78" y="-35.56" rot="R180"/>
+<instance part="LEFTCON" gate="G$1" x="-17.78" y="-35.56" rot="R180"/>
 </instances>
 <busses>
@@
 <wire x1="102.362" y1="1.27" x2="121.412" y2="1.27" width="0.1524" layer="91"/>
 <junction x="102.362" y="1.27"/>
-<pinref part="LEFT" gate="G$1" pin="1"/>
+<pinref part="LEFTCON" gate="G$1" pin="1"/>
 <wire x1="-25.4" y1="-27.94" x2="-25.4" y2="0" width="0.1524" layer="91"/>
 <wire x1="-25.4" y1="0" x2="28.702" y2="1.27" width="0.1524" layer="91"/>
@@
 <wire x1="11.938" y1="-46.228" x2="-27.94" y2="-53.34" width="0.1524" layer="91"/>
 <junction x="11.938" y="-46.228"/>
-<pinref part="LEFT" gate="G$1" pin="3"/>
+<pinref part="LEFTCON" gate="G$1" pin="3"/>
 <wire x1="-25.4" y1="-30.48" x2="-27.94" y2="-30.48" width="0.1524" layer="91"/>
 <wire x1="-27.94" y1="-30.48" x2="-27.94" y2="-53.34" width="0.1524" layer="91"/>
@@
 <junction x="16.764" y="-84.328"/>
 <wire x1="-30.48" y1="-86.36" x2="-30.48" y2="-33.02" width="0.1524" layer="91"/>
-<pinref part="LEFT" gate="G$1" pin="5"/>
+<pinref part="LEFTCON" gate="G$1" pin="5"/>
 <wire x1="-25.4" y1="-33.02" x2="-30.48" y2="-33.02" width="0.1524" layer="91"/>
 <label x="127" y="-83.82" size="1.778" layer="91" xref="yes"/>
@@
 <junction x="19.05" y="-122.428"/>
 <wire x1="-33.02" y1="-35.56" x2="-33.02" y2="-101.6" width="0.1524" layer="91"/>
-<pinref part="LEFT" gate="G$1" pin="7"/>
+<pinref part="LEFTCON" gate="G$1" pin="7"/>
 <wire x1="-25.4" y1="-35.56" x2="-33.02" y2="-35.56" width="0.1524" layer="91"/>
 <wire x1="-33.02" y1="-121.92" x2="-33.02" y2="-101.6" width="0.1524" layer="91"/>
@@
 <wire x1="107.188" y1="-160.528" x2="126.238" y2="-160.528" width="0.1524" layer="91"/>
 <junction x="107.188" y="-160.528"/>
-<pinref part="LEFT" gate="G$1" pin="9"/>
+<pinref part="LEFTCON" gate="G$1" pin="9"/>
 <wire x1="-25.4" y1="-38.1" x2="-35.56" y2="-38.1" width="0.1524" layer="91"/>
 <wire x1="-35.56" y1="-38.1" x2="-35.56" y2="-160.02" width="0.1524" layer="91"/>
@@
 <junction x="16.764" y="-198.628"/>
 <wire x1="-38.1" y1="-198.12" x2="-38.1" y2="-40.64" width="0.1524" layer="91"/>
-<pinref part="LEFT" gate="G$1" pin="11"/>
+<pinref part="LEFTCON" gate="G$1" pin="11"/>
 <wire x1="-38.1" y1="-40.64" x2="-25.4" y2="-40.64" width="0.1524" layer="91"/>
 <label x="116.84" y="-198.12" size="1.778" layer="91" xref="yes"/>
@@
 <wire x1="8.89" y1="-178.308" x2="4.064" y2="-216.408" width="0.1524" layer="91"/>
 <junction x="8.89" y="-178.308"/>
-<pinref part="LEFT" gate="G$1" pin="2"/>
+<pinref part="LEFTCON" gate="G$1" pin="2"/>
 <wire x1="-10.16" y1="-27.94" x2="-2.54" y2="-27.94" width="0.1524" layer="91"/>
 <wire x1="-2.54" y1="-27.94" x2="-0.762" y2="-64.008" width="0.1524" layer="91"/>
@@
 <wire x1="108.712" y1="-102.108" x2="94.488" y2="-64.008" width="0.1524" layer="91"/>
 <junction x="108.712" y="-102.108"/>
-<pinref part="LEFT" gate="G$1" pin="12"/>
+<pinref part="LEFTCON" gate="G$1" pin="12"/>
 <wire x1="-10.16" y1="-40.64" x2="93.98" y2="-40.64" width="0.1524" layer="91"/>
 <pinref part="F3" gate="G$1" pin="P0"/>
@@
 <net name="COL3" class="0">
 <segment>
-<pinref part="LEFT" gate="G$1" pin="6"/>
+<pinref part="LEFTCON" gate="G$1" pin="6"/>
 <wire x1="-10.16" y1="-33.02" x2="35.56" y2="-33.02" width="0.1524" layer="91"/>
 <pinref part="COMMAND" gate="G$1" pin="P0"/>
@@
 <net name="COL7" class="0">
 <segment>
-<pinref part="LEFT" gate="G$1" pin="14"/>
+<pinref part="LEFTCON" gate="G$1" pin="14"/>
 <wire x1="-10.16" y1="-43.18" x2="114.3" y2="-43.18" width="0.1524" layer="91"/>
 <pinref part="F4" gate="G$1" pin="P0"/>
@@
 <net name="COL2" class="0">
 <segment>
-<pinref part="LEFT" gate="G$1" pin="4"/>
+<pinref part="LEFTCON" gate="G$1" pin="4"/>
 <wire x1="-10.16" y1="-30.48" x2="15.24" y2="-30.48" width="0.1524" layer="91"/>
 <pinref part="OPTION" gate="G$1" pin="P0"/>
@@
 <net name="COL5" class="0">
 <segment>
-<pinref part="LEFT" gate="G$1" pin="10"/>
+<pinref part="LEFTCON" gate="G$1" pin="10"/>
 <wire x1="-10.16" y1="-38.1" x2="73.66" y2="-38.1" width="0.1524" layer="91"/>
 <pinref part="F2" gate="G$1" pin="P0"/>
@@
 <net name="COL4" class="0">
 <segment>
-<pinref part="LEFT" gate="G$1" pin="8"/>
+<pinref part="LEFTCON" gate="G$1" pin="8"/>
 <wire x1="-10.16" y1="-35.56" x2="53.34" y2="-35.56" width="0.1524" layer="91"/>
 <pinref part="F1" gate="G$1" pin="P0"/>
