File: eagle/nek-type-a/center.brd (EAGLE design)
At the start: 55 x 70 mm, 8 parts, among them IC1 MCP23017SP

Commit message: logo
Parts:
- IC1: value MCP23017SP -> MCP23017E-S/P

Commit message: center rev 001
Parts:
- renumbered POWER to SWITCH
Connections:
- net N$1 renamed RESET
Routing:
- net GND: track 26.7 -> 29.9 mm
Changed lines of the file:
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@@
 <hole x="50" y="5" drill="3.2"/>
 <hole x="5" y="5" drill="3.2"/>
-<hole x="25" y="65" drill="3.2"/>
+<hole x="27.5" y="65" drill="3.2"/>
 <text x="54.5" y="1" size="1.4224" layer="25" rot="R90">NEK Type A Center - © 2018 Mike Roberts - Revision 001</text>
 <wire x1="24.573790625" y1="47.4066" x2="24.573790625" y2="51.57325" width="0.5" layer="25"/>
@@
 <elements>
 <element name="IC1" library="adafruit" package="DIL28-3" value="MCP23017E-S/P" x="7" y="51" smashed="yes" rot="R90">
-<attribute name="VALUE" x="7.9398" y="35.252" size="1.778" layer="27" ratio="10" rot="R90"/>
+<attribute name="VALUE" x="7.9398" y="35.252" size="1.778" layer="25" ratio="10" rot="R90"/>
 </element>
 <element name="LCON" library="con-harting" library_urn="urn:adsk.eagle:library:151" package="CON14" package3d_urn="urn:adsk.eagle:package:7117/1" value="LCON" x="35.6" y="9.99" rot="R180">
@@
 </element>
 <element name="MS1" library="adafruit" package="FEATHERWING_DIM" value="FEATHERWING_NODIM" x="29.5" y="69.27" rot="R270"/>
-<element name="POWER" library="adafruit" package="JST-PH-2-THM" value="SWITCH" x="16.85" y="64.96" rot="R90"/>
-<element name="R1" library="Seeed-Resistor" library_urn="urn:adsk.eagle:library:474" package="PR-D2.3XL6.5MM" package3d_urn="urn:adsk.eagle:package:32794/1" value="4.7K" x="23" y="32" rot="R180">
+<element name="SWITCH" library="adafruit" package="JST-PH-2-THM" value="SWITCH" x="16.85" y="64.96" rot="R90"/>
+<element name="R1" library="Seeed-Resistor" library_urn="urn:adsk.eagle:library:474" package="PR-D2.3XL6.5MM" package3d_urn="urn:adsk.eagle:package:32794/1" value="4.7K" x="23" y="32" smashed="yes" rot="R180">
 <attribute name="MPN" value="FHCFR-1/4W-472J" x="23" y="32" size="1.778" layer="27" rot="R180" display="off"/>
+<attribute name="NAME" x="25.413" y="30.603" size="0.889" layer="25" ratio="11" rot="R180"/>
+<attribute name="VALUE" x="25.413" y="34.921" size="0.889" layer="25" ratio="11" rot="R180"/>
 </element>
-<element name="R2" library="Seeed-Resistor" library_urn="urn:adsk.eagle:library:474" package="PR-D2.3XL6.5MM" package3d_urn="urn:adsk.eagle:package:32794/1" value="4.7K" x="23" y="26" rot="R180">
+<element name="R2" library="Seeed-Resistor" library_urn="urn:adsk.eagle:library:474" package="PR-D2.3XL6.5MM" package3d_urn="urn:adsk.eagle:package:32794/1" value="4.7K" x="23" y="26" smashed="yes" rot="R180">
 <attribute name="MPN" value="FHCFR-1/4W-472J" x="23" y="26" size="1.778" layer="27" rot="R180" display="off"/>
+<attribute name="NAME" x="25.413" y="24.603" size="0.889" layer="25" ratio="11" rot="R180"/>
+<attribute name="VALUE" x="25.413" y="28.921" size="0.889" layer="25" ratio="11" rot="R180"/>
 </element>
-<element name="R3" library="Seeed-Resistor" library_urn="urn:adsk.eagle:library:474" package="PR-D2.3XL6.5MM" package3d_urn="urn:adsk.eagle:package:32794/1" value="4.7K" x="23" y="20" rot="R180">
+<element name="R3" library="Seeed-Resistor" library_urn="urn:adsk.eagle:library:474" package="PR-D2.3XL6.5MM" package3d_urn="urn:adsk.eagle:package:32794/1" value="4.7K" x="23" y="20" smashed="yes" rot="R180">
 <attribute name="MPN" value="FHCFR-1/4W-472J" x="23" y="20" size="1.778" layer="27" rot="R180" display="off"/>
+<attribute name="NAME" x="25.413" y="18.603" size="0.889" layer="25" ratio="11" rot="R180"/>
+<attribute name="VALUE" x="25.413" y="22.921" size="0.889" layer="25" ratio="11" rot="R180"/>
 </element>
 <element name="RCON" library="con-harting" library_urn="urn:adsk.eagle:library:151" package="CON20" package3d_urn="urn:adsk.eagle:package:7115/1" value="RCON" x="10.79" y="16.75" smashed="yes" rot="R90">
@@
 <wire x1="52.324" y1="26.67" x2="51.308" y2="25.654" width="0.254" layer="16"/>
 <wire x1="52.324" y1="53.34" x2="52.324" y2="26.67" width="0.254" layer="16"/>
-<wire x1="41.402" y1="64.262" x2="52.324" y2="53.34" width="0.254" layer="16"/>
-<wire x1="27.432" y1="64.262" x2="41.402" y2="64.262" width="0.254" layer="16"/>
-<wire x1="25.908" y1="62.738" x2="27.432" y2="64.262" width="0.254" layer="16"/>
-<wire x1="12.954" y1="62.738" x2="25.908" y2="62.738" width="0.254" layer="16"/>
+<wire x1="42.926" y1="62.738" x2="52.324" y2="53.34" width="0.254" layer="16"/>
 <wire x1="10.922" y1="64.77" x2="12.954" y2="62.738" width="0.254" layer="16"/>
 <wire x1="51.308" y1="24.892" x2="51.09" y2="24.82" width="0.254" layer="16"/>
 <wire x1="10.922" y1="64.77" x2="10.81" y2="64.97" width="0.254" layer="16"/>
+<wire x1="12.954" y1="62.738" x2="28.311321875" y2="62.738" width="0.254" layer="16"/>
+<wire x1="28.311321875" y1="62.738" x2="29.8355375" y2="64.262215625" width="0.254" layer="16"/>
+<wire x1="29.8355375" y1="64.262215625" x2="41.401784375" y2="64.262215625" width="0.254" layer="16"/>
+<wire x1="41.401784375" y1="64.262215625" x2="42.926" y2="62.738" width="0.254" layer="16"/>
 </signal>
 <signal name="GND">
 <contactref element="IC1" pad="10"/>
 <contactref element="MS1" pad="4"/>
-<contactref element="POWER" pad="2"/>
-<wire x1="10.922" y1="57.912" x2="10.922" y2="57.404" width="0.254" layer="1"/>
-<wire x1="16.764" y1="63.754" x2="10.922" y2="57.912" width="0.254" layer="1"/>
-<wire x1="10.922" y1="57.404" x2="10.81" y2="57.35" width="0.254" layer="1"/>
-<wire x1="16.764" y1="63.754" x2="16.85" y2="63.96" width="0.254" layer="1"/>
-<wire x1="25.4" y1="55.372" x2="30.734" y2="55.372" width="0.254" layer="1"/>
-<wire x1="17.018" y1="63.754" x2="25.4" y2="55.372" width="0.254" layer="1"/>
+<contactref element="SWITCH" pad="2"/>
+<wire x1="25.4" y1="55.372" x2="30.734" y2="55.372" width="0.5" layer="1"/>
 <wire x1="30.734" y1="55.372" x2="30.77" y2="55.3" width="0.254" layer="1"/>
-<wire x1="17.018" y1="63.754" x2="16.85" y2="63.96" width="0.254" layer="1"/>
+<wire x1="10.81" y1="57.35" x2="16.85" y2="63.39" width="0.5" layer="1"/>
+<wire x1="16.85" y1="63.39" x2="16.85" y2="63.96" width="0.5" layer="1"/>
+<wire x1="25.4" y1="55.372" x2="12.788" y2="55.372" width="0.5" layer="1"/>
+<wire x1="12.788" y1="55.372" x2="10.81" y2="57.35" width="0.5" layer="1"/>
 </signal>
 <signal name="ROW2">
@@
 <contactref element="IC1" pad="16"/>
 <contactref element="IC1" pad="17"/>
-<wire x1="27.94" y1="25.908" x2="27.94" y2="20.066" width="0.254" layer="1"/>
+<wire x1="27.94" y1="25.908" x2="27.94" y2="20.066" width="0.5" layer="1"/>
 <wire x1="27.94" y1="20.066" x2="27.953" y2="20" width="0.254" layer="1"/>
 <wire x1="27.94" y1="25.908" x2="27.953" y2="26" width="0.254" layer="1"/>
-<wire x1="27.94" y1="26.162" x2="27.94" y2="31.75" width="0.254" layer="1"/>
+<wire x1="27.94" y1="26.162" x2="27.94" y2="31.75" width="0.5" layer="1"/>
 <wire x1="27.94" y1="31.75" x2="27.953" y2="32" width="0.254" layer="1"/>
 <wire x1="27.94" y1="26.162" x2="27.953" y2="26" width="0.254" layer="1"/>
-<wire x1="3.302" y1="64.77" x2="3.302" y2="62.484" width="0.254" layer="1"/>
+<wire x1="3.302" y1="64.77" x2="3.302" y2="62.484" width="0.5" layer="1"/>
 <wire x1="3.302" y1="62.484" x2="3.19" y2="62.43" width="0.254" layer="1"/>
 <wire x1="3.302" y1="64.77" x2="3.19" y2="64.97" width="0.254" layer="1"/>
-<wire x1="3.302" y1="62.23" x2="10.668" y2="54.864" width="0.254" layer="1"/>
+<wire x1="3.302" y1="62.23" x2="10.668" y2="54.864" width="0.5" layer="1"/>
 <wire x1="10.668" y1="54.864" x2="10.81" y2="54.81" width="0.254" layer="1"/>
 <wire x1="3.302" y1="62.23" x2="3.19" y2="62.43" width="0.254" layer="1"/>
-<wire x1="3.302" y1="65.024" x2="3.302" y2="67.31" width="0.254" layer="1"/>
+<wire x1="3.302" y1="65.024" x2="3.302" y2="67.31" width="0.5" layer="1"/>
 <wire x1="3.302" y1="67.31" x2="3.19" y2="67.51" width="0.254" layer="1"/>
 <wire x1="3.302" y1="65.024" x2="3.19" y2="64.97" width="0.254" layer="1"/>
-<wire x1="16.256" y1="60.198" x2="27.94" y2="60.198" width="0.254" layer="16"/>
-<wire x1="27.94" y1="60.198" x2="30.734" y2="60.198" width="0.254" layer="16"/>
-<wire x1="10.922" y1="54.864" x2="16.256" y2="60.198" width="0.254" layer="16"/>
+<wire x1="16.256" y1="60.198" x2="27.94" y2="60.198" width="0.5" layer="16"/>
+<wire x1="27.94" y1="60.198" x2="30.734" y2="60.198" width="0.5" layer="16"/>
+<wire x1="10.922" y1="54.864" x2="16.256" y2="60.198" width="0.5" layer="16"/>
 <wire x1="30.734" y1="60.198" x2="30.77" y2="60.38" width="0.254" layer="16"/>
 <wire x1="10.922" y1="54.864" x2="10.81" y2="54.81" width="0.254" layer="16"/>
-<wire x1="27.94" y1="60.198" x2="27.94" y2="32.004" width="0.254" layer="16"/>
+<wire x1="27.94" y1="60.198" x2="27.94" y2="32.004" width="0.5" layer="16"/>
 <wire x1="27.94" y1="32.004" x2="27.953" y2="32" width="0.254" layer="16"/>
 </signal>
@@
 <wire x1="12.192" y1="28.194" x2="12.06" y2="28.18" width="0.254" layer="1"/>
 </signal>
-<signal name="N$1">
+<signal name="RESET">
 <contactref element="IC1" pad="18"/>
 <contactref element="R3" pad="2"/>
@@
 </signal>
 <signal name="EN">
-<contactref element="POWER" pad="1"/>
+<contactref element="SWITCH" pad="1"/>
 <contactref element="MS1" pad="27"/>
 <wire x1="22.86" y1="66.04" x2="17.018" y2="66.04" width="0.254" layer="1"/>

Commit message: center rev 2
Parts:
- R1, R2, R3: value 4.7K -> 4K7
- SWITCH: device adafruit:JST-PH-2-THM -> Rembrandt Electronics - JST XH Connectors v1-0:JST-XH-02-PACKAGE-LONG-PAD
- moved LCON 1.60 mm to (34.0, 9.99)
- moved RCON 1.46 mm to (12.2, 16.8)
- moved SWITCH 0.65 mm to (17.5, 65.0)
Connections:
- net EN: now also SWITCH.2; no longer SWITCH.1
- net GND: now also SWITCH.1; no longer SWITCH.2
Routing:
- net ROW4: track 75.9 -> 63.6 mm
- net LCOL4: track 35.2 -> 43.3 mm
- net LCOL5: track 46.8 -> 39.4 mm
- net ROW1: track 81.2 -> 86.8 mm
- net SDA: track 120.8 -> 116.9 mm
- net RCOL4: track 35.3 -> 39.2 mm
- net ROW5: track 57.7 -> 54.2 mm
- net ROW2: track 85.4 -> 81.9 mm
- net ROW6: track 49.6 -> 46.3 mm
- net ROW3: track 76.5 -> 78.3 mm
- net SCL: track 112.9 -> 114.4 mm
- net EN: track 41.9 -> 42.8 mm
- net LCOL6: track 42.4 -> 43.2 mm
- net GND: track 29.9 -> 29.2 mm
- net LCOL7: track 19.8 -> 20.4 mm
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Other:
- board text added: "NEK Type A Center - © 2018 Mike Roberts - Revision 002"
- board text removed: "NEK Type A Center - © 2018 Mike Roberts - Revision 001"
