File: eagle/nek-type-a/center.sch (EAGLE design)
At the start: 8 parts, among them IC1 MCP23017SP

Commit message: logo
Parts:
- IC1: value MCP23017SP -> MCP23017E-S/P
Changed lines of the file:
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@@
 <part name="LCON" library="con-harting" library_urn="urn:adsk.eagle:library:151" deviceset="CON14" device="" package3d_urn="urn:adsk.eagle:package:7117/1" value="LCON"/>
 <part name="RCON" library="con-harting" library_urn="urn:adsk.eagle:library:151" deviceset="CON20" device="" package3d_urn="urn:adsk.eagle:package:7115/1" value="RCON"/>
-<part name="IC1" library="adafruit" deviceset="MCP23017" device="SP"/>
+<part name="IC1" library="adafruit" deviceset="MCP23017" device="SP" value="MCP23017E-S/P"/>
 <part name="R1" library="Seeed-Resistor" library_urn="urn:adsk.eagle:library:474" deviceset="DIP-RES-4.7K-5%-1/4W(PR-D2.3XL6.5MM)" device="" package3d_urn="urn:adsk.eagle:package:32794/1" value="4.7K"/>
 <part name="R2" library="Seeed-Resistor" library_urn="urn:adsk.eagle:library:474" deviceset="DIP-RES-4.7K-5%-1/4W(PR-D2.3XL6.5MM)" device="" package3d_urn="urn:adsk.eagle:package:32794/1" value="4.7K"/>

Commit message: center rev 001
Parts:
- renumbered POWER to SWITCH
Connections:
- net N$1 renamed RESET
Changed lines of the file:
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@@
 <part name="R2" library="Seeed-Resistor" library_urn="urn:adsk.eagle:library:474" deviceset="DIP-RES-4.7K-5%-1/4W(PR-D2.3XL6.5MM)" device="" package3d_urn="urn:adsk.eagle:package:32794/1" value="4.7K"/>
 <part name="R3" library="Seeed-Resistor" library_urn="urn:adsk.eagle:library:474" deviceset="DIP-RES-4.7K-5%-1/4W(PR-D2.3XL6.5MM)" device="" package3d_urn="urn:adsk.eagle:package:32794/1" value="4.7K"/>
-<part name="POWER" library="adafruit" deviceset="JST_2PIN" device="-THM" value="SWITCH"/>
+<part name="SWITCH" library="adafruit" deviceset="JST_2PIN" device="-THM" value="SWITCH"/>
 </parts>
 <sheets>
@@
 <instance part="R2" gate="G$1" x="48.26" y="40.64"/>
 <instance part="R3" gate="G$1" x="38.1" y="50.8"/>
-<instance part="POWER" gate="G$1" x="43.18" y="25.4"/>
+<instance part="SWITCH" gate="G$1" x="43.18" y="25.4"/>
 </instances>
 <busses>
@@
 <wire x1="43.18" y1="-25.4" x2="43.18" y2="-33.02" width="0.1524" layer="91"/>
 <wire x1="43.18" y1="-33.02" x2="25.4" y2="-33.02" width="0.1524" layer="91"/>
-<pinref part="POWER" gate="G$1" pin="1"/>
+<pinref part="SWITCH" gate="G$1" pin="1"/>
 <wire x1="40.64" y1="27.94" x2="25.4" y2="27.94" width="0.1524" layer="91"/>
 <junction x="25.4" y="27.94"/>
@@
 </segment>
 </net>
-<net name="N$1" class="0">
+<net name="RESET" class="0">
 <segment>
 <pinref part="IC1" gate="G$1" pin="!RESET"/>
@@
 <net name="EN" class="0">
 <segment>
-<pinref part="POWER" gate="G$1" pin="2"/>
+<pinref part="SWITCH" gate="G$1" pin="2"/>
 <wire x1="40.64" y1="25.4" x2="40.64" y2="20.32" width="0.1524" layer="91"/>
 <wire x1="40.64" y1="20.32" x2="48.26" y2="20.32" width="0.1524" layer="91"/>

Commit message: center rev 2
Parts:
- R1, R2, R3: value 4.7K -> 4K7
- SWITCH: device adafruit:JST_2PIN-THM -> Rembrandt Electronics - JST XH Connectors v1-0:JST-XH-02-PIN-LONG-PAD
Connections:
- net EN: now also SWITCH-2.S; no longer SWITCH.2
- net GND: now also SWITCH-1.S; no longer SWITCH.1
Changed lines of the file:
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@@
 <part name="RCON" library="con-harting" library_urn="urn:adsk.eagle:library:151" deviceset="CON20" device="" package3d_urn="urn:adsk.eagle:package:7115/1" value="RCON"/>
 <part name="IC1" library="adafruit" deviceset="MCP23017" device="SP" value="MCP23017E-S/P"/>
-<part name="R1" library="Seeed-Resistor" library_urn="urn:adsk.eagle:library:474" deviceset="DIP-RES-4.7K-5%-1/4W(PR-D2.3XL6.5MM)" device="" package3d_urn="urn:adsk.eagle:package:32794/1" value="4.7K"/>
-<part name="R2" library="Seeed-Resistor" library_urn="urn:adsk.eagle:library:474" deviceset="DIP-RES-4.7K-5%-1/4W(PR-D2.3XL6.5MM)" device="" package3d_urn="urn:adsk.eagle:package:32794/1" value="4.7K"/>
-<part name="R3" library="Seeed-Resistor" library_urn="urn:adsk.eagle:library:474" deviceset="DIP-RES-4.7K-5%-1/4W(PR-D2.3XL6.5MM)" device="" package3d_urn="urn:adsk.eagle:package:32794/1" value="4.7K"/>
-<part name="SWITCH" library="adafruit" deviceset="JST_2PIN" device="-THM" value="SWITCH"/>
+<part name="R1" library="Seeed-Resistor" library_urn="urn:adsk.eagle:library:474" deviceset="DIP-RES-4.7K-5%-1/4W(PR-D2.3XL6.5MM)" device="" package3d_urn="urn:adsk.eagle:package:32794/1" value="4K7"/>
+<part name="R2" library="Seeed-Resistor" library_urn="urn:adsk.eagle:library:474" deviceset="DIP-RES-4.7K-5%-1/4W(PR-D2.3XL6.5MM)" device="" package3d_urn="urn:adsk.eagle:package:32794/1" value="4K7"/>
+<part name="R3" library="Seeed-Resistor" library_urn="urn:adsk.eagle:library:474" deviceset="DIP-RES-4.7K-5%-1/4W(PR-D2.3XL6.5MM)" device="" package3d_urn="urn:adsk.eagle:package:32794/1" value="4K7"/>
+<part name="SWITCH" library="Rembrandt Electronics - JST XH Connectors v1-0" deviceset="JST-XH-02-PIN" device="-LONG-PAD" value="SWITCH"/>
 </parts>
 <sheets>
@@
 <instance part="R2" gate="G$1" x="48.26" y="40.64"/>
 <instance part="R3" gate="G$1" x="38.1" y="50.8"/>
-<instance part="SWITCH" gate="G$1" x="43.18" y="25.4"/>
+<instance part="SWITCH" gate="-2" x="43.18" y="25.4"/>
+<instance part="SWITCH" gate="-1" x="43.18" y="27.94"/>
 </instances>
 <busses>
@@
 <wire x1="43.18" y1="-25.4" x2="43.18" y2="-33.02" width="0.1524" layer="91"/>
 <wire x1="43.18" y1="-33.02" x2="25.4" y2="-33.02" width="0.1524" layer="91"/>
-<pinref part="SWITCH" gate="G$1" pin="1"/>
 <wire x1="40.64" y1="27.94" x2="25.4" y2="27.94" width="0.1524" layer="91"/>
 <junction x="25.4" y="27.94"/>
+<pinref part="SWITCH" gate="-1" pin="S"/>
 </segment>
 </net>
@@
 <net name="EN" class="0">
 <segment>
-<pinref part="SWITCH" gate="G$1" pin="2"/>
 <wire x1="40.64" y1="25.4" x2="40.64" y2="20.32" width="0.1524" layer="91"/>
 <wire x1="40.64" y1="20.32" x2="48.26" y2="20.32" width="0.1524" layer="91"/>
 <pinref part="MS1" gate="G$1" pin="EN"/>
 <wire x1="48.26" y1="20.32" x2="48.26" y2="17.78" width="0.1524" layer="91"/>
-</segment>
-</net>
+<pinref part="SWITCH" gate="-2" pin="S"/>
+</segment>
+</net>
